Commit message: new update

File: description/gazebo_control.xacro (robot description, xacro)
@@ -12,8 +12,8 @@
             <max_wheel_acceleration>10.0</max_wheel_acceleration>
             <!--Output-->
-            <odometry_frame>odam</odometry_frame>
+            <odometry_frame>odom</odometry_frame>
             <robot_base_frame>base_link</robot_base_frame>
-            <publish_odam>true</publish_odam>
-            <publish_odam_tf>true</publish_odam_tf>
+            <publish_odom>true</publish_odom>
+            <publish_odom_tf>true</publish_odom_tf>
             <publish_wheel_tf>true</publish_wheel_tf>
         </plugin>

File: description/robot.urdf.xacro (robot description, xacro)
@@ -3,3 +3,4 @@
     <xacro:include filename="robot_core.xacro" />
     <xacro:include filename="gazebo_control.xacro" />
+    <xacro:include filename="lidar.xacro" />
 </robot>

File: description/robot_core.xacro (robot description, xacro)
@@ -13,4 +13,7 @@
     <material name="black">
         <color rgba="0 0 0 1"/>
+    </material>
+    <material name="red">
+        <color rgba="1 0 0 1"/>
     </material>
     <!-- Base Link -->
